File: MULTIGW.kicad_sch (KiCad schematic)
At the start: 32 parts, among them J1 HR911105A, J2 Conn_01x06_Male, J3 Power, U1 AMS1117-3.3, U2 ESP32-WROOM-32, U3 LAN8720A

Commit message: Small tidy up
Parts:
- J2: value Conn_01x06_Male -> (none)
Other:
- note added: "3.3V LDO"
- note added: "Connectors"
- note added: "Ethernet connector"
- note added: "MCU"
- note added: "PHY"
- moved on the sheet: C1, C10, C11, C2, C3, C4, C6, C7, C8, C9, D1, J1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
